File: hw/sch_pcb/AIRDOS04_base/power.kicad_sch (KiCad schematic)
At the start: 9 parts, among them U4 TPS613222ADBV

Commit message: Change analog supply voltage to 5V. Change ADC reference to 4.1V.
Parts:
- added C50: 10uF, Capacitor_Tantalum_SMD:CP_EIA-3216-18_Kemet-A, symbol Device:C_Polarized_Small
- added C59: 100nF, Capacitor_SMD:C_0805_2012Metric, symbol Device:C
- added U3: ISL21080DIH309, Package_TO_SOT_SMD:SOT-23, symbol Reference_Voltage:ISL21070CIH320Z-TK
Connections:
- net +5V: now also C50.1
- net GNDA: now also C50.2, C59.2, U3.3 (GND)
- net VCC: now also C59.1, U3.1 (Vin)
- new net REF: U3.2 (Vout)
Other:
- note added: "REF 0.9 V is the lowest value of reasonably available voltage reference."

Commit message: Fix path to kicad workflow. Add submodule to battery module.
Other:
- company: (none) -> Jakub Kákona <info@ust.cz>
- title: (none) -> AIRDOS04A base board
Changed lines of the file:
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@@
 (kicad_sch (version 20230121) (generator eeschema)
   (paper "A4")
+  (title_block
+    (title "AIRDOS04A base board")
+    (date "2023-10-23")
+    (company "Jakub Kákona <info@ust.cz>")
+    (comment 2 "Airborne semiconductor\\nradiation detector")
+  )
   (junction (at 204.47 60.96) (diameter 0) (color 0 0 0 0)
   )
